File: pcb/releasebuttonboard.sch (KiCad schematic (older format))
At the start: 24 parts, among them U1 24C16, U2 RASPIPLUSHEADER, U3 OLEDHeader, U4 REncHeader, U5 BtnHeader, U6 PAM8407

Commit message: Schematic for extra rotary encoder PCB.
Parts:
- added SW?: ROTENC, symbol ROTENC
- added U?: RENCHEADER, symbol RENCHEADER
Connections:
- wire segments 123 -> 143
Other:
- note added: "ROTARY ENCODER PCB"
Changed lines of the file:
@@
 Text Notes 3550 900  2    60   ~ 0
 RASPBERRY PI A/B+\nGPIO HEADER
+$Comp
+L RENCHEADER U?
+U 1 1 54A8BB2E
+P 9450 5900
+F 0 "U?" H 9450 6250 60  0000 C CNN
+F 1 "RENCHEADER" H 9650 5600 60  0000 C CNN
+F 2 "" H 9450 5950 60  0000 C CNN
+F 3 "" H 9450 5950 60  0000 C CNN
+	1    9450 5900
+	0    1    1    0
+$EndComp
+$Comp
+L ROTENC SW?
+U 1 1 54A8BB42
+P 9450 5300
+F 0 "SW?" H 9350 5500 60  0000 C CNN
+F 1 "ROTENC" H 9650 5100 60  0000 R CNN
+F 2 "" H 9400 5300 60  0000 C CNN
+F 3 "" H 9400 5300 60  0000 C CNN
+	1    9450 5300
+	-1   0    0    1
+$EndComp
+Wire Wire Line
+	8950 5350 8900 5350
+Wire Wire Line
+	8900 5350 8900 5550
+Wire Wire Line
+	8900 5550 9350 5550
+Wire Wire Line
+	9350 5550 9350 5900
+Wire Wire Line
+	9250 5900 9250 5650
+Wire Wire Line
+	9250 5650 8800 5650
+Wire Wire Line
+	8800 5650 8800 5250
+Wire Wire Line
+	8800 5250 8950 5250
+Wire Wire Line
+	9500 5900 9500 5550
+Wire Wire Line
+	9500 5550 10000 5550
+Wire Wire Line
+	10000 5550 10000 5400
+Wire Wire Line
+	10000 5400 9950 5400
+Wire Wire Line
+	9600 5900 9600 5650
+Wire Wire Line
+	9600 5650 10100 5650
+Wire Wire Line
+	10100 5650 10100 5300
+Wire Wire Line
+	10100 5300 9950 5300
+Wire Wire Line
+	9700 5900 9700 5750
+Wire Wire Line
+	9700 5750 10200 5750
+Wire Wire Line
+	10200 5750 10200 5200
+Wire Wire Line
+	10200 5200 9950 5200
+Text Notes 9800 5000 2    60   ~ 0
+ROTARY ENCODER PCB
+Wire Notes Line
+	8700 4850 8700 6500
+Wire Notes Line
+	8700 6500 10300 6500
+Wire Notes Line
+	10300 6500 10300 4850
+Wire Notes Line
+	10300 4850 8700 4850
 $EndSCHEMATC

Commit message: More schematic annotation.
Parts:
- gave numbers to parts that had none: 2
Changed lines of the file:
@@
 RASPBERRY PI A/B+\nGPIO HEADER
 $Comp
-L RENCHEADER U?
+L RENCHEADER U7
 U 1 1 54A8BB2E
 P 9450 5900
-F 0 "U?" H 9450 6250 60  0000 C CNN
+F 0 "U7" H 9450 6250 60  0000 C CNN
 F 1 "RENCHEADER" H 9650 5600 60  0000 C CNN
 F 2 "" H 9450 5950 60  0000 C CNN
@@
 $EndComp
 $Comp
-L ROTENC SW?
+L ROTENC SW1
 U 1 1 54A8BB42
 P 9450 5300
-F 0 "SW?" H 9350 5500 60  0000 C CNN
+F 0 "SW1" H 9350 5500 60  0000 C CNN
 F 1 "ROTENC" H 9650 5100 60  0000 R CNN
 F 2 "" H 9400 5300 60  0000 C CNN

Commit message: Fix rotary encoder header schematic reference.
It seems that the case sensitivity rules change when moving between KiCad
versions.
Parts:
- removed U7: RENCHEADER, symbol RENCHEADER
- added U7: REncHeader, symbol REncHeader
Changed lines of the file:
@@
 LIBS:releasebutton
 LIBS:releasebuttonboard-cache
-EELAYER 24 0
+EELAYER 25 0
 EELAYER END
 $Descr USLetter 11000 8500
@@
 RASPBERRY PI A/B+\nGPIO HEADER
 $Comp
-L RENCHEADER U7
-U 1 1 54A8BB2E
-P 9450 5900
-F 0 "U7" H 9450 6250 60  0000 C CNN
-F 1 "RENCHEADER" H 9650 5600 60  0000 C CNN
-F 2 "" H 9450 5950 60  0000 C CNN
-F 3 "" H 9450 5950 60  0000 C CNN
-	1    9450 5900
-	0    1    1    0
-$EndComp
-$Comp
 L ROTENC SW1
 U 1 1 54A8BB42
@@
 	8900 5550 9350 5550
 Wire Wire Line
-	9350 5550 9350 5900
-Wire Wire Line
-	9250 5900 9250 5650
-Wire Wire Line
 	9250 5650 8800 5650
 Wire Wire Line
@@
 	8800 5250 8950 5250
 Wire Wire Line
-	9500 5900 9500 5550
-Wire Wire Line
 	9500 5550 10000 5550
 Wire Wire Line
@@
 	10000 5400 9950 5400
 Wire Wire Line
-	9600 5900 9600 5650
-Wire Wire Line
 	9600 5650 10100 5650
 Wire Wire Line
@@
 Wire Wire Line
 	10100 5300 9950 5300
-Wire Wire Line
-	9700 5900 9700 5750
 Wire Wire Line
 	9700 5750 10200 5750
@@
 Wire Notes Line
 	10300 4850 8700 4850
+$Comp
+L REncHeader U7
+U 1 1 54A8C599
+P 9450 5900
+F 0 "U7" H 9450 6250 60  0000 C CNN
+F 1 "REncHeader" H 9650 5600 60  0000 C CNN
+F 2 "" H 9450 5950 60  0000 C CNN
+F 3 "" H 9450 5950 60  0000 C CNN
+	1    9450 5900
+	0    1    1    0
+$EndComp
+Wire Wire Line
+	9250 5900 9250 5650
+Wire Wire Line
+	9350 5550 9350 5900
+Wire Wire Line
+	9500 5900 9500 5550
+Wire Wire Line
+	9600 5900 9600 5650
+Wire Wire Line
+	9700 5900 9700 5750
 $EndSCHEMATC
