File: pcb/releasebuttonboard.sch (KiCad schematic (older format))
At the start: 26 parts, among them SW1 ROTENC, U1 24C16, U2 RASPIPLUSHEADER, U3 OLEDHeader, U4 REncHeader, U5 BtnHeader, U6 PAM8407, U7 REncHeader

Commit message: Power the audio amp from the 5V supply.
This should keep it a little more isolated from the digital supply as well
as making it easier to route the power tracks.
Connections:
- net VCC: no longer C6.1, C7.2, R4.1, U6.16 (VDD), U6.4 (UP), U6.5 (DOWN), U6.9 (VDD)
- net AVCC: now reaches U2.2 (+5V)
- net AVCC: now also C6.1, C7.2, R4.1, U2.4 (+5V), U6.16 (VDD), U6.4 (UP), U6.5 (DOWN), U6.9 (VDD)
Changed lines of the file:
@@
 $EndComp
 Text GLabel 9950 850  2    60   Input ~ 0
-VCC
+AVCC
 Text GLabel 9950 2050 2    60   Input ~ 0
 GND
@@
 $EndComp
 Text GLabel 9950 3250 2    60   Input ~ 0
-VCC
+AVCC
 $Comp
 L C C6
@@
 $EndComp
 Text GLabel 5150 2050 0    60   Input ~ 0
-VCC
+AVCC
 $Comp
 L R R4
@@
 Wire Wire Line
 	2350 3400 2400 3400
+Text GLabel 1000 1500 3    60   Output ~ 0
+AVCC
+Wire Wire Line
+	1050 1350 1000 1350
+Wire Wire Line
+	1000 1350 1000 1500
+Wire Wire Line
+	1050 1450 1000 1450
+Connection ~ 1000 1450
 $EndSCHEMATC
